Commit message: Add collision and inertia to AMR model, spawn it in Gazebo

File: src/warehouse_description/urdf/warehouse_amr.urdf.xacro (robot description, xacro)
@@ -13,8 +13,35 @@
   <xacro:property name="lidar_radius" value="0.04"/>
   <xacro:property name="lidar_length" value="0.05"/>
-  <!-- Colours, defined once and reused by name -->
+  <!-- Colours-->
   <material name="orange"><color rgba="1.0 0.5 0.1 1.0"/></material>
   <material name="black"><color rgba="0.1 0.1 0.1 1.0"/></material>
   <material name="grey"><color rgba="0.6 0.6 0.6 1.0"/></material>
+  <xacro:macro name="box_inertia" params="m x y z xyz rpy">
+    <inertial>
+      <origin xyz="${xyz}" rpy="${rpy}"/>
+      <mass value="${m}"/>
+      <inertia ixx="${m*(y*y + z*z)/12}" ixy="0" ixz="0"
+               iyy="${m*(x*x + z*z)/12}" iyz="0"
+               izz="${m*(x*x + y*y)/12}"/>
+    </inertial>
+  </xacro:macro>
+  <xacro:macro name="cylinder_inertia" params="m r h xyz rpy">
+    <inertial>
+      <origin xyz="${xyz}" rpy="${rpy}"/>
+      <mass value="${m}"/>
+      <inertia ixx="${m*(3*r*r + h*h)/12}" ixy="0" ixz="0"
+               iyy="${m*(3*r*r + h*h)/12}" iyz="0"
+               izz="${m*r*r/2}"/>
+    </inertial>
+  </xacro:macro>
+  <xacro:macro name="sphere_inertia" params="m r xyz rpy">
+    <inertial>
+      <origin xyz="${xyz}" rpy="${rpy}"/>
+      <mass value="${m}"/>
+      <inertia ixx="${2*m*r*r/5}" ixy="0" ixz="0"
+               iyy="${2*m*r*r/5}" iyz="0"
+               izz="${2*m*r*r/5}"/>
+    </inertial>
+  </xacro:macro>
   <!-- A point on the floor under the robot -->
   <link name="base_footprint"/>
@@ -33,4 +60,12 @@
       <material name="orange"/>
     </visual>
+    <collision>
+      <origin xyz="0 0 ${ground_clearance + base_height/2 - wheel_radius}" rpy="0 0 0"/>
+      <geometry>
+        <box size="${base_length} ${base_width} ${base_height}"/>
+      </geometry>
+    </collision>
+    <xacro:box_inertia m="10" x="${base_length}" y="${base_width}" z="${base_height}"
+                       xyz="0 0 ${ground_clearance + base_height/2 - wheel_radius}" rpy="0 0 0"/>
   </link>
   <!-- Left wheel -->
@@ -43,4 +78,13 @@
       <material name="black"/>
     </visual>
+    <collision>
+      <origin xyz="0 0 0" rpy="${pi/2} 0 0"/>
+      <geometry>
+        <cylinder radius="${wheel_radius}" length="${wheel_width}"/>
+      </geometry>
+    </collision>
+    <!-- left_wheel AND right_wheel (identical) -->
+    <xacro:cylinder_inertia m="0.5" r="${wheel_radius}" h="${wheel_width}"
+                            xyz="0 0 0" rpy="${pi/2} 0 0"/>
   </link>
   <joint name="left_wheel_joint" type="continuous">
@@ -59,4 +103,13 @@
       <material name="black"/>
     </visual>
+    <collision>
+      <origin  xyz="0 0 0" rpy="${pi/2} 0 0"/>
+      <geometry>
+        <cylinder radius="${wheel_radius}" length="${wheel_width}"/>
+      </geometry>
+    </collision>
+    <!-- left_wheel AND right_wheel (identical) -->
+    <xacro:cylinder_inertia m="0.5" r="${wheel_radius}" h="${wheel_width}"
+                            xyz="0 0 0" rpy="${pi/2} 0 0"/>
   </link>
   <joint name="right_wheel_joint" type="continuous">
@@ -75,4 +128,10 @@
       <material name="grey"/>
     </visual>
+    <collision>
+      <geometry>
+        <sphere radius="${caster_radius}"/>
+      </geometry>
+    </collision>
+    <xacro:sphere_inertia m="0.1" r="${caster_radius}" xyz="0 0 0" rpy="0 0 0"/>
   </link>
   <joint name="front_caster_joint" type="fixed">
@@ -90,4 +149,10 @@
       <material name="grey"/>
     </visual>
+    <collision>
+      <geometry>
+        <sphere radius="${caster_radius}"/>
+      </geometry>
+    </collision>
+    <xacro:sphere_inertia m="0.1" r="${caster_radius}" xyz="0 0 0" rpy="0 0 0"/>
   </link>
   <joint name="rear_caster_joint" type="fixed">
@@ -102,6 +167,13 @@
         <cylinder radius="${lidar_radius}" length="${lidar_length}"/>
       </geometry>
-      <material name="red"/>
+      <material name="red" rgba="1.0 0.0 0.0 1.0"/>
     </visual>
+    <collision>
+      <geometry>
+        <cylinder radius="${lidar_radius}" length="${lidar_length}"/>
+      </geometry>
+    </collision>
+    <xacro:cylinder_inertia m="0.2" r="${lidar_radius}" h="${lidar_length}"
+                            xyz="0 0 0" rpy="0 0 0"/>
   </link>
   <joint name="lidar_joint" type="fixed">

Commit message: Tidy up

File: src/warehouse_description/urdf/warehouse_amr.urdf.xacro (robot description, xacro)
@@ -17,4 +17,5 @@
   <material name="black"><color rgba="0.1 0.1 0.1 1.0"/></material>
   <material name="grey"><color rgba="0.6 0.6 0.6 1.0"/></material>
+  <material name="red"><color rgba="1.0 0.0 0.0 1.0"/></material>
   <xacro:macro name="box_inertia" params="m x y z xyz rpy">
     <inertial>
@@ -84,5 +85,5 @@
       </geometry>
     </collision>
-    <!-- left_wheel AND right_wheel (identical) -->
+    <!-- left_wheel-->
     <xacro:cylinder_inertia m="0.5" r="${wheel_radius}" h="${wheel_width}"
                             xyz="0 0 0" rpy="${pi/2} 0 0"/>
@@ -109,5 +110,5 @@
       </geometry>
     </collision>
-    <!-- left_wheel AND right_wheel (identical) -->
+    <!--right_wheel-->
     <xacro:cylinder_inertia m="0.5" r="${wheel_radius}" h="${wheel_width}"
                             xyz="0 0 0" rpy="${pi/2} 0 0"/>
@@ -167,5 +168,5 @@
         <cylinder radius="${lidar_radius}" length="${lidar_length}"/>
       </geometry>
-      <material name="red" rgba="1.0 0.0 0.0 1.0"/>
+      <material name="red"/>
     </visual>
     <collision>
